Commit message: Restored PickNik erroneously removed

File: eli_cs_robot_description/urdf/cs.urdf.xacro (robot description, xacro)
@@ -10,4 +10,5 @@
    <!-- parameters -->
    <xacro:arg name="tf_prefix" default="" />
+   <xacro:arg name="parent" default="world" />
    <xacro:arg name="joint_limit_params" default="$(find eli_cs_robot_description)/config/$(arg cs_type)/joint_limits.yaml"/>
    <xacro:arg name="kinematics_params" default="$(find eli_cs_robot_description)/config/$(arg cs_type)/default_kinematics.yaml"/>
@@ -47,11 +48,15 @@
    <!-- convert to property to use substitution in function -->
    <xacro:property name="initial_positions_file" default="$(arg initial_positions_file)"/>
-   <!-- create link fixed to the "world" -->
-   <link name="world" />
+   <!-- Convert argument into a Xacro variable -->
+   <xacro:property name="parent_var" value="$(arg parent)" />
+   <xacro:if value="${parent_var == 'world'}">
+     <!-- create link fixed to the "world" -->
+     <link name="world" />
+   </xacro:if>
    <!-- arm -->
    <xacro:cs_robot
      name="$(arg name)"
      tf_prefix="$(arg tf_prefix)"
-     parent="world"
+     parent="$(arg parent)"
      joint_limits_parameters_file="$(arg joint_limit_params)"
      kinematics_parameters_file="$(arg kinematics_params)"
@@ -85,5 +90,5 @@
      trajectory_port="$(arg trajectory_port)"
      >
-     <origin xyz="0 0 0" rpy="0 0 0" />          <!-- position robot in the world -->
+     <origin xyz="0 0 0" rpy="0 0 0" />          <!-- position robot in the parent frame -->
    </xacro:cs_robot>
    <xacro:if value="$(arg sim_gazebo)">

File: eli_cs_robot_description/urdf/cs_macro.xacro (robot description, xacro)
@@ -204,9 +204,15 @@
       <xacro:build_inertial mass="${wrist_3_mass}" cog="${prop_wrist_3_cog}" inertia="${prop_wrist_3_inertia}"/>
     </link>
-     <!-- base_joint fixes base_link to the environment -->
+    <link name="fts_link" />
+    <joint name="fts_link_joint" type="fixed">
+      <parent link="${parent}" />
+      <child link="fts_link" />
+      <origin xyz="0.0 0 0.0" rpy="3.14 0 3.14" />
+    </joint>
+    <!-- base_joint fixes base_link to the environment -->
     <joint name="${tf_prefix}base_joint" type="fixed">
-      <xacro:insert_block name="origin" />
-      <parent link="${parent}" />
+      <parent link="fts_link" />
       <child link="${tf_prefix}base_link" />
+      <origin xyz="0.0 0 0.0" rpy="-3.14 0 -3.14" />
     </joint>
     <!-- joints - main serial chain -->
